File: hardware/KungFuFlash2.kicad_pcb (KiCad board)
At the start: 2 copper layers, 62.4 x 62 mm, 52 parts, among them J1 SWD, J2 USB_B_Micro, J3 Wifi, Q1 BC817, SW1 Reset, SW2 Menu, SW3 Special, U1 C64-Exp-Port, U2 AMS1117-3.3, U3 STM32H7B0VBTx, Y1 25 MHz

Commit message: Refining design and updating README.md
Routing:
- net GND: track 659.5 -> 673.3 mm
Other:
- board text added: "Original board design: https://github.com/KimJorgensen/KungFuFlash2 Adaptations: https://github.com/ifilot/kungfu-flash-2"
- board text added: "Rev. 1 / A"
- board text removed: "Board adapted from: https://github.com/KimJorgensen/KungFuFlash2"
- board text removed: "Rev. 1.a"
Changed lines of the file:
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@@
 		(tags "SMD SMT crystal")
 		(property "Reference" "Y1"
-			(at 0 -2.45 270)
+			(at 0 -2.45 -90)
 			(layer "F.SilkS")
 			(effects
@@
 		)
 		(property "Value" "25 MHz"
-			(at 0 2.45 270)
+			(at 0 2.45 -90)
 			(layer "F.Fab")
 			(effects
@@
 		)
 		(fp_text user "${REFERENCE}"
-			(at 0 0 270)
+			(at 0 0 -90)
 			(layer "F.Fab")
 			(effects
@@
 		(tags "capacitor handsolder")
 		(property "Reference" "C16"
-			(at 0.4585 1.524 0)
+			(at -2.3355 1.524 0)
 			(layer "F.SilkS")
 			(effects
@@
 		(layer "Edge.Cuts")
 	)
-	(gr_text "Board adapted from:\nhttps://github.com/KimJorgensen/KungFuFlash2"
-		(at 78.867 79.121 90)
+	(gr_text "Original board design:\nhttps://github.com/KimJorgensen/KungFuFlash2\n\nAdaptations:\nhttps://github.com/ifilot/kungfu-flash-2"
+		(at 81.28 79.121 90)
 		(layer "B.SilkS")
 		(effects
@@
 		)
 	)
-	(gr_text "Rev. 1.a"
-		(at 80.391 96.4184 0)
+	(gr_text "Rev. 1 / A"
+		(at 81.28 96.012 0)
 		(layer "F.SilkS")
 		(effects
@@
 	)
 	(segment
+		(start 131.064 81.116)
+		(end 131.064 83.916)
+		(width 0.25)
+		(layer "F.Cu")
+		(net 1)
+	)
+	(segment
 		(start 122.555 106.934)
 		(end 122.555 111.379)
@@
 	)
 	(segment
+		(start 136.564 89.916)
+		(end 131.064 89.916)
+		(width 0.25)
+		(layer "F.Cu")
+		(net 1)
+	)
+	(segment
 		(start 120.6705 97.967)
 		(end 120.396 97.6925)
@@
 	)
 	(segment
+		(start 136.564 81.116)
+		(end 131.064 81.116)
+		(width 0.25)
+		(layer "F.Cu")
+		(net 1)
+	)
+	(segment
 		(start 116.5352 90.5256)
 		(end 116.078 90.9828)
@@
 	)
 	(segment
-		(start 134.9819 85.1726)
-		(end 135.001 85.1535)
-		(width 0.25)
-		(layer "F.Cu")
-		(net 1)
-	)
-	(segment
 		(start 114.3 78.613)
 		(end 114.935 77.978)
@@
 		(polygon
 			(pts
-				(xy 74.93 67.31) (xy 139.7 67.31) (xy 139.7 123.19) (xy 74.93 123.19)
+				(xy 74.93 67.31) (xy 139.7 67.31) (xy 139.7 121.92) (xy 74.93 121.92)
 			)
 		)
