File: hardware/KungFuFlash2.kicad_sch (KiCad schematic)
At the start: 52 parts, among them J1 SWD, J2 USB_B_Micro, J3 Wifi, Q1 BC817, SW1 Reset, SW2 Menu, SW3 Special, U1 C64-Exp-Port, U2 AMS1117-3.3, U3 STM32H7B0VBTx, Y1 25 MHz

Commit message: Refining design and updating README.md
Parts:
- Q1: LCSC Part # C466643 -> (none)
- XS1: LCSC Part # C91145 -> (none)
Other:
- note added: "Adapted from: https://github.com/KimJorgensen/KungFuFlash2 Small modifications made to increase compatibility with "basic" components of JLCPCB Fab. Sources: https://github.com/ifilot/kungfu-flash-2"
Changed lines of the file:
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@@
 		)
 	)
+	(text "Adapted from: https://github.com/KimJorgensen/KungFuFlash2\nSmall modifications made to increase compatibility with \n\"basic\" components of JLCPCB Fab.\nSources: https://github.com/ifilot/kungfu-flash-2"
+		(exclude_from_sim no)
+		(at 199.898 174.752 0)
+		(effects
+			(font
+				(size 1.27 1.27)
+			)
+			(justify left)
+		)
+	)
 	(label "A0"
 		(at 88.9 138.43 180)
@@
 			)
 		)
-		(property "LCSC Part #" "C91145"
+		(property "LCSC Part #" ""
 			(at 255.27 90.17 0)
 			(effects
@@
 			)
 		)
-		(property "LCSC Part #" "C466643"
+		(property "LCSC Part #" ""
 			(at 198.12 34.29 0)
 			(effects
@@
 			)
 		)
-		(property "Sim.Enable" "0"
-			(at 186.69 173.99 0)
-			(effects
-				(font
-					(size 1.27 1.27)
-				)
-				(hide yes)
-			)
-		)
 		(instances
 			(project "KungFuFlash2"
@@
 	)
 	(symbol
-		(lib_id "power:PWR_FLAG")
-		(at 264.16 25.4 0)
-		(unit 1)
-		(exclude_from_sim no)
-		(in_bom yes)
-		(on_board yes)
-		(dnp no)
-		(fields_autoplaced yes)
-		(property "Reference" "#FLG03"
-			(at 264.16 23.495 0)
-			(effects
-				(font
-					(size 1.27 1.27)
-				)
-				(hide yes)
-			)
-		)
-		(property "Value" "PWR_FLAG"
-			(at 264.16 20.32 0)
-			(effects
-				(font
-					(size 1.27 1.27)
-				)
-			)
-		)
-		(property "Footprint" ""
-			(at 264.16 25.4 0)
-			(effects
-				(font
-					(size 1.27 1.27)
-				)
-				(hide yes)
-			)
-		)
-		(property "Datasheet" "~"
-			(at 264.16 25.4 0)
-			(effects
-				(font
-					(size 1.27 1.27)
-				)
-				(hide yes)
-			)
-		)
-		(property "Description" "Special symbol for telling ERC where power comes from"
-			(at 264.16 25.4 0)
-			(effects
-				(font
-					(size 1.27 1.27)
-				)
-				(hide yes)
-			)
-		)
-		(pin "1"
-		)
-		(instances
-			(project "KungFuFlash2"
-				(path "/900d3ff0-0a04-4b16-beae-b4a6786432f6"
-					(reference "#FLG03")
-					(unit 1)
-				)
-			)
-		)
-	)
-	(symbol
 		(lib_id "power:+3V3")
 		(at 118.11 44.45 0)
@@
 					(unit 1)
 				)
-			)
-		)
-	)
-	(symbol
-		(lib_id "power:+5V")
-		(at 264.16 25.4 180)
-		(unit 1)
-		(exclude_from_sim no)
-		(in_bom yes)
-		(on_board yes)
-		(dnp no)
-		(property "Reference" "#PWR07"
-			(at 264.16 21.59 0)
-			(effects
-				(font
-					(size 1.27 1.27)
-				)
-				(hide yes)
-			)
-		)
-		(property "Value" "+5V"
-			(at 263.779 29.7942 0)
-			(effects
-				(font
-					(size 1.27 1.27)
-				)
-			)
-		)
-		(property "Footprint" ""
-			(at 264.16 25.4 0)
-			(effects
-				(font
-					(size 1.27 1.27)
-				)
-				(hide yes)
-			)
-		)
-		(property "Datasheet" ""
-			(at 264.16 25.4 0)
-			(effects
-				(font
-					(size 1.27 1.27)
-				)
-				(hide yes)
-			)
-		)
-		(property "Description" "Power symbol creates a global label with name \"+5V\""
-			(at 264.16 25.4 0)
-			(effects
-				(font
-					(size 1.27 1.27)
-				)
-				(hide yes)
-			)
-		)
-		(pin "1"
-		)
-		(instances
-			(project "KungFuFlash2"
-				(path "/900d3ff0-0a04-4b16-beae-b4a6786432f6"
-					(reference "#PWR07")
-					(unit 1)
-				)

Commit message: Filling out all components
Parts:
- J1: LCSC Part # (none) -> C466643
- J2: LCSC Part # (none) -> C46391
- SW1, SW2, SW3: LCSC Part # (none) -> C134186
- XS1: LCSC Part # (none) -> C91145
Changed lines of the file:
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@@
 			)
 		)
-		(property "LCSC Part #" ""
+		(property "LCSC Part #" "C91145"
 			(at 255.27 90.17 0)
 			(effects
@@
 			)
 		)
+		(property "LCSC Part #" "C134186"
+			(at 209.55 92.71 0)
+			(effects
+				(font
+					(size 1.27 1.27)
+				)
+				(hide yes)
+			)
+		)
 		(pin "1"
 		)
@@
 			)
 		)
+		(property "LCSC Part #" "C134186"
+			(at 209.55 107.95 0)
+			(effects
+				(font
+					(size 1.27 1.27)
+				)
+				(hide yes)
+			)
+		)
 		(pin "1"
 		)
@@
 			)
 		)
+		(property "LCSC Part #" "C46391"
+			(at 255.27 48.26 0)
+			(effects
+				(font
+					(size 1.27 1.27)
+				)
+				(hide yes)
+			)
+		)
 		(pin "1"
 		)
@@
 			)
 		)
+		(property "LCSC Part #" "C466643"
+			(at 200.66 62.23 0)
+			(effects
+				(font
+					(size 1.27 1.27)
+				)
+				(hide yes)
+			)
+		)
 		(pin "1"
 		)
@@
 			(at 76.2 31.75 0)
 			(effects
+				(font
+					(size 1.27 1.27)
+				)
+				(hide yes)
+			)
+		)
+		(property "LCSC Part #" "C134186"
+			(at 76.2 31.75 0)
+			(effects

Commit message: Fixing wrong component
Parts:
- J1: LCSC Part # C466643 -> (none)
- Q1: LCSC Part # (none) -> C466643
Changed lines of the file:
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@@
 			)
 		)
-		(property "LCSC Part #" ""
+		(property "LCSC Part #" "C466643"
 			(at 198.12 34.29 0)
 			(effects
@@
 			)
 		)
-		(property "LCSC Part #" "C466643"
+		(property "LCSC Part #" ""
 			(at 200.66 62.23 0)
 			(effects
